File: HW2/hw2/hw2.brd (EAGLE design)
At the start: 50 x 50 mm, 22 parts, among them IC1 PIC32MX250F128B, IC2 MCP1702, J1 USB-MB-H, SW1 SLIDE

Commit message: finished wiring board
Parts:
- moved LED1 33.9 mm to (35.6, 3.81), turned to 180 degrees
- moved LED2 33.9 mm to (2.54, 11.4), turned to 0 degrees
- moved R1 18.2 mm to (25.4, 2.54), turned to 0 degrees
- moved R2 18.2 mm to (7.62, 6.35), turned to 90 degrees
- moved C3 3.45 mm to (17.3, 42.9)
- moved C2 2.16 mm to (17.5, 7.62)
- moved IC1 0.46 mm to (25.3, 22.8)
- moved C1 0.25 mm to (32.0, 38.1), turned to 270 degrees
- turned R3 to 180 degrees
- turned RESET to 180 degrees
- flipped SW1 to the bottom
Routing:
- net +3V3: track 0.00 -> 152.3 mm, vias 0 -> 2
- net +5V: track 0.00 -> 76.6 mm, vias 0 -> 2
- net USBID: track 0.00 -> 50.3 mm, vias 0 -> 1
- net B4/USER: track 0.00 -> 45.3 mm
- net D-: track 0.00 -> 38.3 mm, vias 0 -> 1
- net MCLR: track 0.00 -> 37.1 mm
- net D+: track 0.00 -> 35.8 mm, vias 0 -> 1
- net A4/LED: track 0.00 -> 35.3 mm
- net PGC: track 0.00 -> 30.5 mm, vias 0 -> 1
- net PGD: track 0.00 -> 30.5 mm, vias 0 -> 1
- net B9: track 0.00 -> 26.0 mm
- net B8: track 0.00 -> 25.9 mm
- net B7: track 0.00 -> 25.9 mm
- net A0: track 0.00 -> 21.2 mm
- net B2: track 0.00 -> 21.2 mm
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- added copper zone on layer 16, net GND
