File: HW2/hw2/hw2.sch (EAGLE design)
At the start: 22 parts, among them IC1 PIC32MX250F128B, IC2 MCP1702, J1 USB-MB-H, SW1 SLIDE

Commit message: finished wiring board
Other:
- moved on the sheet: C3
Changed lines of the file:
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@@
 <part name="GND4" library="hw2" deviceset="GND" device=""/>
 <part name="GND5" library="hw2" deviceset="GND" device=""/>
-<part name="GND6" library="hw2" deviceset="GND" device=""/>
 <part name="GND7" library="hw2" deviceset="GND" device=""/>
 <part name="GND8" library="hw2" deviceset="GND" device=""/>
@@
 <instance part="C1" gate="G$1" x="78.74" y="68.58"/>
 <instance part="C2" gate="G$1" x="-20.32" y="7.62"/>
-<instance part="C3" gate="G$1" x="55.88" y="116.84"/>
+<instance part="C3" gate="G$1" x="48.26" y="116.84"/>
 <instance part="C4" gate="G$1" x="114.3" y="116.84"/>
 <instance part="C5" gate="G$1" x="81.28" y="27.94"/>
@@
 <instance part="GND4" gate="1" x="81.28" y="17.78"/>
 <instance part="GND5" gate="1" x="71.12" y="22.86"/>
-<instance part="GND6" gate="1" x="68.58" y="63.5"/>
-<instance part="GND7" gate="1" x="78.74" y="58.42"/>
+<instance part="GND7" gate="1" x="71.12" y="63.5"/>
 <instance part="GND8" gate="1" x="106.68" y="55.88"/>
 <instance part="GND9" gate="1" x="0" y="101.6"/>
-<instance part="GND10" gate="1" x="55.88" y="109.22"/>
+<instance part="GND10" gate="1" x="48.26" y="109.22"/>
 <instance part="GND11" gate="1" x="91.44" y="101.6"/>
 <instance part="GND12" gate="1" x="114.3" y="106.68"/>
@@
 <instance part="GND18" gate="1" x="160.02" y="43.18"/>
 <instance part="GND19" gate="1" x="210.82" y="43.18"/>
-<instance part="P+1" gate="1" x="48.26" y="121.92"/>
+<instance part="P+1" gate="1" x="63.5" y="121.92"/>
 <instance part="P+2" gate="1" x="60.96" y="7.62" rot="MR0"/>
-<instance part="+3V1" gate="G$1" x="-25.4" y="12.7"/>
-<instance part="+3V2" gate="G$1" x="86.36" y="73.66" rot="MR0"/>
+<instance part="+3V1" gate="G$1" x="-7.62" y="12.7"/>
+<instance part="+3V2" gate="G$1" x="71.12" y="73.66"/>
 <instance part="+3V3" gate="G$1" x="73.66" y="48.26"/>
 <instance part="+3V4" gate="G$1" x="109.22" y="38.1"/>
@@
 </segment>
 <segment>
-<pinref part="IC1" gate="G$1" pin="27.AVSS"/>
-<wire x1="50.8" y1="66.04" x2="68.58" y2="66.04" width="0.1524" layer="91"/>
-<pinref part="GND6" gate="1" pin="GND"/>
-</segment>
-<segment>
-<pinref part="C1" gate="G$1" pin="2"/>
-<pinref part="GND7" gate="1" pin="GND"/>
-<wire x1="78.74" y1="63.5" x2="78.74" y2="60.96" width="0.1524" layer="91"/>
-</segment>
-<segment>
 <pinref part="IC1" gate="G$1" pin="19.VSS"/>
 <wire x1="50.8" y1="25.4" x2="71.12" y2="25.4" width="0.1524" layer="91"/>
@@
 <wire x1="198.12" y1="45.72" x2="210.82" y2="45.72" width="0.1524" layer="91"/>
 <pinref part="GND19" gate="1" pin="GND"/>
+</segment>
+<segment>
+<pinref part="C1" gate="G$1" pin="2"/>
+<wire x1="78.74" y1="63.5" x2="73.66" y2="63.5" width="0.1524" layer="91"/>
+<wire x1="73.66" y1="63.5" x2="73.66" y2="66.04" width="0.1524" layer="91"/>
+<pinref part="GND7" gate="1" pin="GND"/>
+<wire x1="73.66" y1="66.04" x2="71.12" y2="66.04" width="0.1524" layer="91"/>
+<pinref part="IC1" gate="G$1" pin="27.AVSS"/>
+<wire x1="71.12" y1="66.04" x2="50.8" y2="66.04" width="0.1524" layer="91"/>
+<junction x="71.12" y="66.04"/>
 </segment>
 </net>
@@
 <net name="+5V" class="0">
 <segment>
-<pinref part="SW1" gate="G$1" pin="1"/>
-<wire x1="40.64" y1="124.46" x2="40.64" y2="119.38" width="0.1524" layer="91"/>
-<pinref part="C3" gate="G$1" pin="1"/>
-<wire x1="40.64" y1="119.38" x2="48.26" y2="119.38" width="0.1524" layer="91"/>
-<pinref part="P+1" gate="1" pin="+5V"/>
-<wire x1="48.26" y1="119.38" x2="55.88" y2="119.38" width="0.1524" layer="91"/>
-<junction x="48.26" y="119.38"/>
-<pinref part="IC2" gate="G$1" pin="2.VIN"/>
-<wire x1="55.88" y1="119.38" x2="73.66" y2="119.38" width="0.1524" layer="91"/>
-<junction x="55.88" y="119.38"/>
-</segment>
-<segment>
 <pinref part="IC1" gate="G$1" pin="15.VBUS"/>
 <pinref part="P+2" gate="1" pin="+5V"/>
@@
 <wire x1="198.12" y1="48.26" x2="213.36" y2="48.26" width="0.1524" layer="91"/>
 <pinref part="P+3" gate="1" pin="+5V"/>
+</segment>
+<segment>
+<pinref part="SW1" gate="G$1" pin="1"/>
+<pinref part="IC2" gate="G$1" pin="2.VIN"/>
+<wire x1="40.64" y1="124.46" x2="40.64" y2="119.38" width="0.1524" layer="91"/>
+<wire x1="40.64" y1="119.38" x2="48.26" y2="119.38" width="0.1524" layer="91"/>
+<pinref part="C3" gate="G$1" pin="1"/>
+<wire x1="48.26" y1="119.38" x2="63.5" y2="119.38" width="0.1524" layer="91"/>
+<junction x="48.26" y="119.38"/>
+<pinref part="P+1" gate="1" pin="+5V"/>
+<wire x1="63.5" y1="119.38" x2="73.66" y2="119.38" width="0.1524" layer="91"/>
+<junction x="63.5" y="119.38"/>
 </segment>
 </net>
@@
 </segment>
 <segment>
-<pinref part="+3V1" gate="G$1" pin="+3V3"/>
-<pinref part="C2" gate="G$1" pin="1"/>
-<wire x1="-25.4" y1="10.16" x2="-20.32" y2="10.16" width="0.1524" layer="91"/>
-<pinref part="IC1" gate="G$1" pin="13.VDD"/>
-<wire x1="5.08" y1="10.16" x2="-20.32" y2="10.16" width="0.1524" layer="91"/>
-<junction x="-20.32" y="10.16"/>
-</segment>
-<segment>
-<pinref part="+3V2" gate="G$1" pin="+3V3"/>
-<pinref part="C1" gate="G$1" pin="1"/>
-<wire x1="86.36" y1="71.12" x2="78.74" y2="71.12" width="0.1524" layer="91"/>
-<pinref part="IC1" gate="G$1" pin="28.AVDD"/>
-<wire x1="50.8" y1="71.12" x2="78.74" y2="71.12" width="0.1524" layer="91"/>
-<junction x="78.74" y="71.12"/>
-</segment>
-<segment>
 <pinref part="IC1" gate="G$1" pin="23.VUSB3V3"/>
 <wire x1="50.8" y1="45.72" x2="73.66" y2="45.72" width="0.1524" layer="91"/>
@@
 <pinref part="+3V7" gate="G$1" pin="+3V3"/>
 </segment>
-</net>
+<segment>
+<pinref part="IC1" gate="G$1" pin="28.AVDD"/>
+<pinref part="+3V2" gate="G$1" pin="+3V3"/>
+<wire x1="50.8" y1="71.12" x2="71.12" y2="71.12" width="0.1524" layer="91"/>
+<pinref part="C1" gate="G$1" pin="1"/>
+<wire x1="71.12" y1="71.12" x2="78.74" y2="71.12" width="0.1524" layer="91"/>
+<junction x="71.12" y="71.12"/>
+</segment>
+<segment>
+<pinref part="IC1" gate="G$1" pin="13.VDD"/>
+<pinref part="+3V1" gate="G$1" pin="+3V3"/>
+<wire x1="5.08" y1="10.16" x2="-7.62" y2="10.16" width="0.1524" layer="91"/>
+<pinref part="C2" gate="G$1" pin="1"/>
+<wire x1="-7.62" y1="10.16" x2="-20.32" y2="10.16" width="0.1524" layer="91"/>
+<junction x="-7.62" y="10.16"/>
+</segment>
+</net>

Commit message: updated board with annotations
Parts:
- RESET: value PB -> RESET
- USER: value PB -> USER
Connections:
- net N$14 renamed OSC1
- net N$15 renamed OSC2
Changed lines of the file:
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@@
 <part name="LED1" library="hw2" deviceset="LED" device="3MM" package3d_urn="urn:adsk.eagle:package:15797/1" value="Red"/>
 <part name="LED2" library="hw2" deviceset="LED" device="3MM" package3d_urn="urn:adsk.eagle:package:15797/1" value="Green"/>
-<part name="RESET" library="hw2" deviceset="PB" device=""/>
-<part name="USER" library="hw2" deviceset="PB" device=""/>
+<part name="RESET" library="hw2" deviceset="PB" device="" value="RESET"/>
+<part name="USER" library="hw2" deviceset="PB" device="" value="USER"/>
 <part name="R1" library="hw2" deviceset="R-US_" device="0207/10" package3d_urn="urn:adsk.eagle:package:25939/1" value="330"/>
 <part name="R2" library="hw2" deviceset="R-US_" device="0207/10" package3d_urn="urn:adsk.eagle:package:25939/1" value="330"/>
@@
 </segment>
 </net>
-<net name="N$14" class="0">
+<net name="OSC1" class="0">
 <segment>
 <pinref part="IC1" gate="G$1" pin="9.OSC1/A2"/>
@@
 <wire x1="-10.16" y1="30.48" x2="-12.7" y2="30.48" width="0.1524" layer="91"/>
 <wire x1="-25.4" y1="30.48" x2="-12.7" y2="30.48" width="0.1524" layer="91"/>
-</segment>
-</net>
-<net name="N$15" class="0">
+<label x="-25.4" y="30.48" size="1.778" layer="95"/>
+</segment>
+</net>
+<net name="OSC2" class="0">
 <segment>
 <pinref part="IC1" gate="G$1" pin="10.OSC2/A3"/>
@@
 <wire x1="-25.4" y1="20.32" x2="-17.78" y2="20.32" width="0.1524" layer="91"/>
 <wire x1="-17.78" y1="20.32" x2="-17.78" y2="25.4" width="0.1524" layer="91"/>
-</segment>
-</net>
+<label x="-17.78" y="25.4" size="1.778" layer="95"/>
+</segment>
+</net>
